Commit message: Add_wrist_camera_and_teleoperation_node

File: urdf/armando_camera.urdf.xacro (robot description, xacro)
@@ -41,3 +41,44 @@
         </sensor>
     </gazebo>
+    <!-- ================= 2. NUOVA CAMERA SUL POLSO (END-EFFECTOR) ================= -->
+    <joint name="wrist_camera_joint" type="fixed">
+        <parent link="crawer_base"/>
+        <child link="wrist_camera_link"/>
+        <!-- Posizionata sopra la base della pinza e ruotata per guardare nella direzione di approccio -->
+        <origin xyz="0.0 0.02 0.025" rpy="0 -1.57079632679 1.57079632679"/>
+    </joint>
+    <link name="wrist_camera_link">
+        <visual>
+            <geometry>
+                <box size="0.01 0.02 0.02"/>
+            </geometry>
+            <material name="red"/>
+        </visual>
+    </link>
+    <joint name="wrist_camera_optical_joint" type="fixed">
+        <parent link="wrist_camera_link"/>
+        <child link="wrist_camera_optical_frame"/>
+        <origin xyz="0 0 0" rpy="-1.57079632679 0 -1.57079632679"/>
+    </joint>
+    <link name="wrist_camera_optical_frame"/>
+    <gazebo reference="wrist_camera_link">
+        <sensor name="wrist_camera" type="camera">
+            <camera>
+                <horizontal_fov>1.047</horizontal_fov>
+                <image>
+                    <width>1920</width>
+                    <height>1080</height>
+                </image>
+                <clip>
+                    <near>0.05</near>
+                    <far>5</far>
+                </clip>
+            </camera>
+            <always_on>1</always_on>
+            <update_rate>30</update_rate>
+            <visualize>true</visualize>
+            <topic>wrist_camera</topic>
+            <gz_frame_id>wrist_camera_optical_frame</gz_frame_id>
+        </sensor>
+    </gazebo>
 </robot>
